File: ATmega32U4-breakout_board.kicad_pcb (KiCad board)
At the start: 2 copper layers, 22 parts, among them J1 USB_C_Receptacle_USB2.0_16P, J2 Conn_01x12, J3 Conn_01x12, U2 MIC5219-3.3YM5, U3 ATmega32U4-M, Y1 Crystal_GND24

Commit message: changed pcb v1
Parts:
- C1, C2, C3, C4, C5, C6: footprint Capacitor_SMD:C_0603_1608Metric -> Capacitor_SMD:C_0402_1005Metric
- moved R4 70.3 mm to (129.8, 74.0), turned to 90 degrees
- moved C1 41.6 mm to (154.3, 78.3)
- moved F1 15.7 mm to (133.7, 74.0)
- moved U2 12.1 mm to (138.0, 78.8)
- moved D1 12.0 mm to (137.0, 74.8)
- moved R3 7.95 mm to (139.5, 74.0), turned to 90 degrees
Connections:
- J1 pad A6: Net-(J1-D+-PadA6) -> /D+
- J1 pad A7: Net-(J1-D--PadA7) -> /D-
- J1 pad B6: Net-(J1-D+-PadA6) -> /D+
- J1 pad B7: Net-(J1-D--PadA7) -> /D-
Routing:
- net /RAW: track 0.00 -> 17.8 mm
- net /D-: track 0.00 -> 15.8 mm
- net /D+: track 0.00 -> 15.8 mm
- net +5V: track 0.00 -> 10.1 mm, vias 0 -> 1
- net VCC: track 0.00 -> 8.70 mm
- net Net-(J1-CC1): track 0.00 -> 5.97 mm
- net GND: track 0.00 -> 5.43 mm
- net /D7: track 0.00 -> 3.20 mm
- net Net-(U3-XTAL2): track 0.00 -> 2.26 mm
- net Net-(U3-XTAL1): track 0.00 -> 2.20 mm
- net Net-(J1-CC2): track 0.00 -> 2.11 mm, vias 0 -> 2
- net Net-(D1-A): track 0.00 -> 1.72 mm, vias 0 -> 2
