File: ATmega32U4-breakout_board.kicad_sch (KiCad schematic)
At the start: 20 parts, among them J1 USB_C_Receptacle_USB2.0_16P, U1 ATmega32U4-A, U2 MIC5219-3.3YM5, Y1 Crystal_GND24

Commit message: schematic fix + start of pcb designing
Parts:
- removed U1: ATmega32U4-A, Package_QFP:TQFP-44_10x10mm_P0.8mm, symbol MCU_Microchip_ATmega:ATmega32U4-A
- added J2, J3: Conn_01x12, Connector_PinHeader_2.54mm:PinHeader_1x12_P2.54mm_Vertical, symbol Connector_Generic:Conn_01x12
- added U3: ATmega32U4-M, Package_DFN_QFN:QFN-64-1EP_9x9mm_P0.5mm_EP7.65x7.65mm, symbol MCU_Microchip_ATmega:ATmega32U4-M
- C1: value 1u -> 1uF
- C2, C3: value 22p -> 22pF; footprint (none) -> Capacitor_SMD:C_0603_1608Metric
- C4: value 0.1u -> 0.1uF
- C5: value 1u -> 1uF; footprint (none) -> Capacitor_SMD:C_0603_1608Metric
- C6: value 10u -> 10uF; footprint (none) -> Capacitor_SMD:C_0603_1608Metric
- D1: value D_Schottky -> ~; footprint (none) -> Diode_SMD:D_SOD-123F
- R2, R6: footprint Resistor_SMD:R_0201_0603Metric -> Resistor_SMD:R_0603_1608Metric
- R5: footprint (none) -> Resistor_SMD:R_0603_1608Metric
Connections:
- net D+: now also U3.4 (D+)
- net D-: now also U3.3 (D-)
- net GND: now also Y1.2, Y1.4, J2.3 (Pin_3), J2.4 (Pin_4), J3.2 (Pin_2), U3.15 (GND), U3.23 (GND), U3.35 (GND), U3.43 (GND), U3.45 (GND), U3.5 (UGND)
- net RAW: now also J3.1 (Pin_1)
- net VCC: now also J3.4 (Pin_4), U3.14 (VCC), U3.24 (AVCC), U3.34 (VCC), U3.44 (AVCC)
- net RESET: now reaches R6.2
- net RESET: now also J3.3 (Pin_3), U3.13 (~{RESET})
- net at C3.2, Y1.1: now also U3.16 (XTAL2)
- net at C2.2, Y1.3: now also U3.17 (XTAL1)
- net at C1.1: now also U3.6 (UCAP)
- net VBUS renamed +5V
- net +5V: now also U3.2 (UVCC), U3.7 (VBUS)
- new net B1: J3.9 (Pin_9), U3.9 (PB1)
- new net B2: J3.11 (Pin_11), U3.10 (PB2)
- new net B3: J3.10 (Pin_10), U3.11 (PB3)
- new net B4: J2.11 (Pin_11), U3.28 (PB4)
- new net B5: J2.12 (Pin_12), U3.29 (PB5)
- new net B6: J3.12 (Pin_12), U3.30 (PB6)
- new net C6: J2.8 (Pin_8), U3.31 (PC6)
- new net D0: J2.6 (Pin_6), U3.18 (PD0)
- new net D1: J2.5 (Pin_5), U3.19 (PD1)
- new net D2: J2.2 (Pin_2), U3.20 (PD2)
- new net D3: J2.1 (Pin_1), U3.21 (PD3)
- new net D4: J2.7 (Pin_7), U3.25 (PD4)
- new net D7: J2.9 (Pin_9), U3.27 (PD7)
- new net E6: J2.10 (Pin_10), U3.1 (PE6)
- new net F4: J3.5 (Pin_5), U3.39 (PF4)
- new net F5: J3.6 (Pin_6), U3.38 (PF5)
- new net F6: J3.7 (Pin_7), U3.37 (PF6)
- new net F7: J3.8 (Pin_8), U3.36 (PF7)
- no-connect marks 0 -> 13
Other:
- note added: "Rozmiary footprintow rezystorow i kondensatorow"
- note added: "Wersja Atmegi"
- note added: "Wybranie modeli rezystorow i kondensatorow"
- note removed: "Policzyc czy na pewno 22pf"
- moved on the sheet: C4, C6, D2, R5

Commit message: changed pcb v1
Parts:
- C1, C2, C3, C4, C5, C6: footprint Capacitor_SMD:C_0603_1608Metric -> Capacitor_SMD:C_0402_1005Metric
Changed lines of the file:
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@@
 			)
 		)
-		(property "Footprint" "Capacitor_SMD:C_0603_1608Metric"
+		(property "Footprint" "Capacitor_SMD:C_0402_1005Metric"
 			(at 76.2 125.73 0)
 			(effects
@@
 			)
 		)
-		(property "Footprint" "Capacitor_SMD:C_0603_1608Metric"
+		(property "Footprint" "Capacitor_SMD:C_0402_1005Metric"
 			(at 93.98 125.73 0)
 			(effects
@@
 			)
 		)
-		(property "Footprint" "Capacitor_SMD:C_0603_1608Metric"
+		(property "Footprint" "Capacitor_SMD:C_0402_1005Metric"
 			(at 207.01 88.9 0)
 			(effects
@@
 			)
 		)
-		(property "Footprint" "Capacitor_SMD:C_0603_1608Metric"
+		(property "Footprint" "Capacitor_SMD:C_0402_1005Metric"
 			(at 85.09 125.73 0)
 			(effects
@@
 			)
 		)
-		(property "Footprint" "Capacitor_SMD:C_0603_1608Metric"
+		(property "Footprint" "Capacitor_SMD:C_0402_1005Metric"
 			(at 193.04 64.77 0)
 			(effects
@@
 			)
 		)
-		(property "Footprint" "Capacitor_SMD:C_0603_1608Metric"
+		(property "Footprint" "Capacitor_SMD:C_0402_1005Metric"
 			(at 193.04 57.15 0)
 			(effects
